File: WalletRadio_v2/WalletRadio_v2.kicad_pcb (KiCad board)
At the start: 2 copper layers, 92.3 x 52.8 mm, 45 parts, among them J1 UJC-HP-3-SMT-TR, Q1 DMP212LQ-7, Q2 Q_NPN_ECB, SW1 SW_SPDT, SW2 CUS-13TB, U1 MCP73831-2-OT, U2 Si4824, U3 AZV321KTR-G1

Commit message: Moved some stuff. Also added a graphic
Parts:
- added G***: LOGO, LOGO, F.Cu at (121.4, 102.6)
- moved TP3 19.6 mm to (143.8, 108.5)
- moved TP4 19.5 mm to (141.5, 98.3)
- moved TP2 9.32 mm to (157.2, 106.2)
- moved D3 3.12 mm to (153.4, 103.9), turned to 180 degrees
- moved C6 1.14 mm to (149.9, 102.1)
Routing:
- net Net-(C7-Pad1): track 29.5 -> 8.58 mm, vias 2 -> 0
- net Net-(Q2-Pad3): track 41.3 -> 26.2 mm
- net /+Vbat: track 37.7 -> 40.4 mm, vias 5 -> 6
- net Net-(Q1-Pad2): track 23.2 -> 21.8 mm
- net Net-(C6-Pad1): track 15.0 -> 13.8 mm
- net Net-(R6-Pad2): track 74.7 -> 75.6 mm
Other:
- board text added: "Calvin Field 2022"
- board text added: "SW/AM/FM"
